Commit message: Add the gripper end effector

File: template_project/panda_arm.urdf (robot description, URDF)
Before this commit: robot panda, 8 links, 7 joints
Links:
- added link leftfinger, mass 0.1; visual mesh filename=../../../model/panda/meshes/visual/finger.obj
- added link rightfinger, mass 0.1; visual mesh filename=../../../model/panda/meshes/visual/finger.obj
- link link7: mass 0.5 -> 1.8; geometry visual mesh filename=../../../model/panda/meshes/visual/hand.obj; visual mesh filename=../../../model/panda/meshes/visual/link7.obj
Joints:
- added joint finger_joint1: type prismatic, parent link7, child leftfinger, origin xyz=0 0 0.1654 rpy=0 0 -0.78539816339, axis 0 1 0, limit lower=0.0 upper=0.04 effort=20 velocity=0.2
- added joint finger_joint2: type prismatic, parent link7, child rightfinger, origin xyz=0 0 0.1654 rpy=0 0 -0.78539816339, axis 0 1 0, limit lower=0.0 upper=0.04 effort=20 velocity=0.2
